File: pathfinderKey-Cuts.kicad_pcb (KiCad board)
At the start: 2 copper layers, 10 parts, among them SW1 SW_Push, SW2 SW_Push, SW3 SW_Push, U1 XIAO-RP2040-DIP

Commit message: Add files via upload
Parts:
- added D4: L08R5000Q1, footprints:LEDRD254W57D500H1070, F.Cu at (199.5, 110.5)
- added R4: R, Resistor_THT:R_Axial_DIN0204_L3.6mm_D1.6mm_P5.08mm_Horizontal, F.Cu at (195.0, 107.9)
- added SW4: SW_Push, Button_Switch_Keyboard:SW_Cherry_MX_1.00u_PCB, F.Cu at (201.5, 118.9)
- moved SW3 72.8 mm to (175.0, 118.9)
- moved SW1 72.3 mm to (175.0, 91.9)
- moved SW2 63.1 mm to (201.5, 91.9)
- moved D1 58.0 mm to (173.2, 83.5)
- moved D3 57.5 mm to (173.2, 110.5)
- moved D2 48.0 mm to (199.7, 83.5)
- moved R1 47.8 mm to (168.5, 80.9), turned to -90 degrees
- moved R3 47.4 mm to (168.4, 107.9)
- moved R2 36.5 mm to (195.0, 80.9)
- moved U1 18.4 mm to (149.5, 121.4)
Connections:
- U1 pad 4: LED1 -> button4
- U1 pad 5: LED2 -> LED1
- U1 pad 6: LED3 -> LED2
- U1 pad 7: unconnected-(U1-GPIO0/TX-Pad7) -> LED3
- U1 pad 8: unconnected-(U1-GPIO1/RX-Pad8) -> LED4
Routing:
- net button4: track 0.00 -> 206.5 mm
- net button2: track 33.3 -> 149.7 mm
- net LED2: track 49.1 -> 163.3 mm
- net LED4: track 0.00 -> 102.1 mm
- net LED3: track 9.33 -> 88.7 mm
- net GND: track 174.4 -> 161.7 mm
- net LED1: track 72.0 -> 60.4 mm
- net button3: track 26.7 -> 36.4 mm
- net Net-(D4-PadA): track 0.00 -> 9.04 mm
- net button1: track 42.1 -> 47.9 mm
- net Net-(D3-PadA): track 5.03 -> 7.15 mm
- net Net-(D1-PadA): track 5.50 -> 7.07 mm
Other:
- board outline added: 78 x 60.5 mm
