File: pathfinderKey-Cuts.kicad_pcb (KiCad board)
At the start: 2 copper layers, 81 x 71 mm, 13 parts, among them SW1 SW_Push, SW2 SW_Push, SW3 SW_Push, SW4 SW_Push, U1 XIAO-RP2040-DIP

Commit message: Add files via upload
Routing:
- net LED2: track 152.7 -> 157.4 mm
- net LED1: track 147.5 -> 151.4 mm
- net button1: track 115.8 -> 114.2 mm
- net button2: track 57.3 -> 58.9 mm
- net button3: track 74.2 -> 72.7 mm
