File: pathfinderKey-Cuts.kicad_pcb (KiCad board)
At the start: 2 copper layers, 81 x 71 mm, 13 parts, among them SW1 SW_Push, SW2 SW_Push, SW3 SW_Push, SW4 SW_Push, U1 XIAO-RP2040-DIP

Commit message: Add files via upload
Other:
- board text removed: "?"
