File: pathfinderKey-Cuts.kicad_sch (KiCad schematic)
At the start: 10 parts, among them SW1 SW_Push, SW2 SW_Push, SW3 SW_Push, U1 XIAO-RP2040-DIP

Commit message: Add files via upload
Parts:
- D1, D2, D3: footprint L08R5000Q1:LEDRD254W57D500H1070 -> footprints:LEDRD254W57D500H1070
- SW1, SW2, SW3: footprint (none) -> Button_Switch_Keyboard:SW_Cherry_MX_1.00u_PCB
- U1: footprint Module:MOUDLE14P-XIAO-DIP-SMD -> footprints:XIAO-RP2040-DIP
Changed lines of the file:
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@@
 			)
 		)
-		(property "Footprint" "L08R5000Q1:LEDRD254W57D500H1070"
+		(property "Footprint" "footprints:LEDRD254W57D500H1070"
 			(at 172.72 80.01 0)
 			(effects
@@
 			)
 		)
-		(property "Footprint" "Module:MOUDLE14P-XIAO-DIP-SMD"
+		(property "Footprint" "footprints:XIAO-RP2040-DIP"
 			(at 149.098 141.478 0)
 			(effects
@@
 			)
 		)
-		(property "Footprint" ""
+		(property "Footprint" "Button_Switch_Keyboard:SW_Cherry_MX_1.00u_PCB"
 			(at 119.38 52.07 0)
 			(effects
@@
 			)
 		)
-		(property "Footprint" ""
+		(property "Footprint" "Button_Switch_Keyboard:SW_Cherry_MX_1.00u_PCB"
 			(at 146.05 52.07 0)
 			(effects
@@
 			)
 		)
-		(property "Footprint" ""
+		(property "Footprint" "Button_Switch_Keyboard:SW_Cherry_MX_1.00u_PCB"
 			(at 172.72 52.07 0)
 			(effects
@@
 			)
 		)
-		(property "Footprint" "L08R5000Q1:LEDRD254W57D500H1070"
+		(property "Footprint" "footprints:LEDRD254W57D500H1070"
 			(at 120.65 80.01 0)
 			(effects
@@
 			)
 		)
-		(property "Footprint" "L08R5000Q1:LEDRD254W57D500H1070"
+		(property "Footprint" "footprints:LEDRD254W57D500H1070"
 			(at 146.05 80.01 0)
 			(effects

Commit message: Add files via upload
Parts:
- added D4: L08R5000Q1, footprints:LEDRD254W57D500H1070, symbol L08R5000Q1:L08R5000Q1
- added R4: R, Resistor_THT:R_Axial_DIN0204_L3.6mm_D1.6mm_P5.08mm_Horizontal, symbol Device:R
- added SW4: SW_Push, Button_Switch_Keyboard:SW_Cherry_MX_1.00u_PCB, symbol Switch:SW_Push
Connections:
- net GND: now also D4.C, SW4.2
- net LED1: now also U1.5 (GPIO6/SDA); no longer U1.4 (GPIO29/ADC3/A3)
- net LED2: now also U1.6 (GPIO7/SCL); no longer U1.5 (GPIO6/SDA)
- net LED3: now also U1.7 (GPIO0/TX); no longer U1.6 (GPIO7/SCL)
- net LED4: now reaches U1.8 (GPIO1/RX)
- net LED4: now also R4.2
- new net: D4.A, R4.1
- new net button4: SW4.1, U1.4 (GPIO29/ADC3/A3)
